File: PCB/clackintosh.kicad_pcb (KiCad board)
At the start: 2 copper layers, 325.5 x 155.3 mm, 190 parts, among them SW1 RotaryEncoder_Switch_MP, SW2 SW_SPDT, U1 MCP23017_SP, U2 Nice_Nano_V2

Commit message: final files
Parts:
- added C10: C, Capacitor_THT:CP_Radial_D5.0mm_P2.50mm, B.Cu at (211.5, 93.5)
- added C11: C, Capacitor_THT:CP_Radial_D5.0mm_P2.50mm, B.Cu at (268.6, 93.4)
- added C12: C, Capacitor_THT:CP_Radial_D5.0mm_P2.50mm, B.Cu at (235.4, 112.6)
- added C13: C, Capacitor_THT:CP_Radial_D5.0mm_P2.50mm, B.Cu at (158.7, 112.8)
- added C14: C, Capacitor_THT:CP_Radial_D5.0mm_P2.50mm, B.Cu at (33.5, 130.9)
- added C15: C, Capacitor_THT:CP_Radial_D5.0mm_P2.50mm, B.Cu at (128.4, 143.4)
- added C16: C, Capacitor_THT:CP_Radial_D5.0mm_P2.50mm, B.Cu at (189.9, 139.1)
- added C17: C, Capacitor_THT:CP_Radial_D5.0mm_P2.50mm, B.Cu at (282.2, 145.4)
- added C18: C, Capacitor_THT:CP_Radial_D5.0mm_P2.50mm, B.Cu at (336.3, 123.3)
- added C19: C, Capacitor_THT:CP_Radial_D5.0mm_P2.50mm, B.Cu at (320.9, 59.5)
- added C2: C, Capacitor_THT:CP_Radial_D5.0mm_P2.50mm, B.Cu at (118.5, 53.9)
- added C20: C, Capacitor_THT:CP_Radial_D5.0mm_P2.50mm, B.Cu at (320.5, 95.5)
- added C21: C, Capacitor_THT:CP_Radial_D5.0mm_P2.50mm, F.Cu at (66.6, 19.1)
- added C3: C, Capacitor_THT:CP_Radial_D5.0mm_P2.50mm, B.Cu at (197.3, 53.5)
- added C4: C, Capacitor_THT:CP_Radial_D5.0mm_P2.50mm, B.Cu at (279.2, 53.7)
- added C5: C, Capacitor_THT:CP_Radial_D5.0mm_P2.50mm, B.Cu at (239.9, 74.6)
- added C6: C, Capacitor_THT:CP_Radial_D5.0mm_P2.50mm, B.Cu at (163.7, 74.7)
- added C7: C, Capacitor_THT:CP_Radial_D5.0mm_P2.50mm, B.Cu at (68.3, 74.6)
- added C8: C, Capacitor_THT:CP_Radial_D5.0mm_P2.50mm, B.Cu at (34.2, 94.4)
- added C9: C, Capacitor_THT:CP_Radial_D5.0mm_P2.50mm, B.Cu at (115.9, 93.7)
- C1: moved to B.Cu
- L1, L10, L11, L12, L13, L14, L15, L16, L17, L18, L19, L2, L20, L3, L4, L5, L6, L7, L8, L9: value LED_SK6812MINI -> SK6812MINI-E; footprint LED_SMD:LED_SK6812MINI_PLCC4_3.5x3.5mm_P1.75mm -> sk6812mini-e:MX SK6812MINI E (1); moved to F.Cu
- moved C1 203.5 mm to (36.0, 53.7), turned to 180 degrees
- moved L12 198.1 mm to (253.0, 107.7), turned to 0 degrees
- moved L20 197.7 mm to (319.1, 97.8), turned to 0 degrees
- moved L13 196.8 mm to (174.1, 108.3), turned to 0 degrees
- moved SW2 180.4 mm to (279.3, 19.5)
- moved R2 178.5 mm to (144.3, 23.4), turned to 180 degrees
- moved D59 175.1 mm to (69.2, 124.3)
- moved D57 174.2 mm to (311.7, 104.9)
- moved U2 173.9 mm to (42.2, 18.7)
- moved BT1 173.9 mm to (321.7, 16.9)
- moved D28 173.7 mm to (313.1, 66.7)
- moved D15 173.5 mm to (48.1, 66.9)
- moved D16 173.5 mm to (67.2, 66.9)
- moved D17 173.5 mm to (86.2, 66.9)
- moved D18 173.5 mm to (105.2, 66.9)
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Connections:
- L11 pad 4: Net-(L11-DIN) -> Net-(L10-DOUT)
- L12 pad 4: Net-(L10-DOUT) -> Net-(L11-DOUT)
- L13 pad 4: Net-(L11-DOUT) -> Net-(L12-DOUT)
- L14 pad 4: Net-(L12-DOUT) -> Net-(L13-DOUT)
- L15 pad 4: Net-(L13-DOUT) -> Net-(L14-DOUT)
- L16 pad 2: unconnected-(L16-DOUT-Pad2) -> Net-(L16-DOUT)
- L16 pad 4: Net-(L14-DOUT) -> Net-(L15-DOUT)
- L17 pad 2: unconnected-(L17-DOUT-Pad2) -> Net-(L17-DOUT)
- L17 pad 4: Net-(L15-DOUT) -> Net-(L16-DOUT)
- L18 pad 4: unconnected-(L18-DIN-Pad4) -> Net-(L17-DOUT)
- L2 pad 4: Net-(L2-DIN) -> Net-(L1-DOUT)
- L20 pad 2: Net-(L2-DIN) -> unconnected-(L20-DOUT-Pad2)
- L3 pad 4: Net-(L1-DOUT) -> Net-(L2-DOUT)
- L4 pad 4: Net-(L2-DOUT) -> Net-(L3-DOUT)
- L5 pad 4: Net-(L3-DOUT) -> Net-(L4-DOUT)
- L6 pad 4: Net-(L4-DOUT) -> Net-(L5-DOUT)
- L7 pad 4: Net-(L5-DOUT) -> Net-(L6-DOUT)
- L8 pad 2: Net-(L10-DIN) -> Net-(L8-DOUT)
- L8 pad 4: Net-(L6-DOUT) -> Net-(L7-DOUT)
- L9 pad 2: Net-(L11-DIN) -> Net-(L10-DIN)
- L9 pad 4: Net-(L7-DOUT) -> Net-(L8-DOUT)
Routing:
- net VCC: track 1020.6 -> 1282.4 mm, vias 17 -> 19
- net RE_SW_2: track 1159.6 -> 1387.2 mm, vias 12 -> 22
- net Net-(L2-DIN): track 219.4 -> 0.00 mm, vias 2 -> 0
- net Net-(L11-DIN): track 153.2 -> 0.00 mm, vias 2 -> 0
- net Net-(L11-DOUT): track 172.9 -> 46.4 mm
- net Net-(L4-DOUT): track 155.0 -> 46.3 mm
- net Net-(L5-DOUT): track 175.9 -> 74.8 mm
- net Net-(L14-DOUT): track 160.3 -> 64.7 mm
- net Net-(L16-DOUT): track 0.00 -> 94.4 mm, vias 0 -> 2
- net Net-(L8-DOUT): track 0.00 -> 90.7 mm, vias 0 -> 2
- net Net-(L2-DOUT): track 162.4 -> 93.1 mm
- net Net-(L1-DOUT): track 159.7 -> 91.4 mm
- net Net-(L13-DOUT): track 49.1 -> 114.8 mm
- net Net-(L15-DOUT): track 166.1 -> 105.8 mm
- net Net-(L12-DOUT): track 126.3 -> 78.2 mm
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Other:
- board size 325.5 x 155.3 mm -> 326.2 x 155.4 mm

Commit message: after-review updates
Parts:
- R1, R2: value Resistor_1.8kohm -> Resistor_4.7kohm
- moved C16 23.6 mm to (213.3, 142.0)
- moved C19 5.72 mm to (321.4, 65.2)
- moved C2 5.11 mm to (123.6, 53.8)
- moved C3 4.61 mm to (201.9, 53.4)
Routing:
- net RE_SW_2: track 1387.2 -> 1394.0 mm
- net VCC: track 1282.4 -> 1278.9 mm, vias 19 -> 18
Other:
- board text added: "CLACKINTOSH"
