File: PCB/clackintosh.kicad_sch (KiCad schematic)
At the start: 8 parts, among them SW1 RotaryEncoder_Switch_MP, SW2 SW_SPDT, U1 MCP23017_SP, U2 Nice_Nano_V2

Commit message: final files
Parts:
- renumbered C1 to C21
Changed lines of the file:
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@@
 		(dnp no)
 		(fields_autoplaced yes)
-		(property "Reference" "C1"
+		(property "Reference" "C21"
 			(at 109.22 134.6199 0)
 			(effects
@@
 			(project ""
 				(path "/fb760b86-a9c3-4bd1-911b-58540f9e772a"
-					(reference "C1")
+					(reference "C21")
 					(unit 1)
 				)

Commit message: after-review updates
Parts:
- R1, R2: value Resistor_1.8kohm -> Resistor_4.7kohm
Other:
- note added: "100nF"
Changed lines of the file:
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@@
+		)
+	)
+	(text "100nF\n"
+		(exclude_from_sim no)
+		(at 111.76 139.7 0)
+		(effects
+			(font
+				(size 1.27 1.27)
+			)
 		)
 	)
@@
 			)
 		)
-		(property "Value" "Resistor_1.8kohm"
+		(property "Value" "Resistor_4.7kohm"
 			(at 120.904 109.22 90)
 			(effects
@@
 			)
 		)
-		(property "Value" "Resistor_1.8kohm"
+		(property "Value" "Resistor_4.7kohm"
 			(at 119.888 94.234 90)
 			(effects
