File: PCB/neopixels.kicad_sch (KiCad schematic)
At the start: 20 parts

Commit message: final files
Parts:
- removed L1, L10, L11, L12, L13, L14, L15, L16, L17, L18, L19, L2, L20, L3, L4, L5, L6, L7, L8, L9: LED_SK6812MINI, LED_SMD:LED_SK6812MINI_PLCC4_3.5x3.5mm_P1.75mm, symbol ScottoKeebs:LED_SK6812MINI
- added C1, C10, C11, C12, C13, C14, C15, C16, C17, C18, C19, C2, C20, C3, C4, C5, C6, C7, C8, C9: C, Capacitor_THT:CP_Radial_D5.0mm_P2.50mm, symbol Device:C
- added L1, L10, L11, L12, L13, L14, L15, L16, L17, L18, L19, L2, L20, L3, L4, L5, L6, L7, L8, L9: SK6812MINI-E, sk6812mini-e:MX SK6812MINI E (1), symbol KiCad Keyboard Parts:SK6812MINI-E
Connections:
- net GND: now also C1.2, C10.2, C11.2, C12.2, C13.2, C14.2, C15.2, C16.2, C17.2, C18.2, C19.2, C2.2, C20.2, C3.2, C4.2, C5.2, C6.2, C7.2, C8.2, C9.2, L1.3 (VSS), L10.3 (VSS), L11.3 (VSS), L12.3 (VSS), L13.3 (VSS), L14.3 (VSS), L15.3 (VSS), L16.3 (VSS), L17.3 (VSS), L18.3 (VSS), L19.3 (VSS), L2.3 (VSS), L20.3 (VSS), L3.3 (VSS), L4.3 (VSS), L5.3 (VSS), L6.3 (VSS), L7.3 (VSS), L8.3 (VSS), L9.3 (VSS)
- net LED: now also L1.4 (DIN)
- net VCC: now also C1.1, C10.1, C11.1, C12.1, C13.1, C14.1, C15.1, C16.1, C17.1, C18.1, C19.1, C2.1, C20.1, C3.1, C4.1, C5.1, C6.1, C7.1, C8.1, C9.1, L1.1 (VDD), L10.1 (VDD), L11.1 (VDD), L12.1 (VDD), L13.1 (VDD), L14.1 (VDD), L15.1 (VDD), L16.1 (VDD), L17.1 (VDD), L18.1 (VDD), L19.1 (VDD), L2.1 (VDD), L20.1 (VDD), L3.1 (VDD), L4.1 (VDD), L5.1 (VDD), L6.1 (VDD), L7.1 (VDD), L8.1 (VDD), L9.1 (VDD)
- new net: L17.2 (DOUT), L18.4 (DIN)
- new net: L16.2 (DOUT), L17.4 (DIN)
- new net: L1.2 (DOUT), L2.4 (DIN)
- new net: L10.2 (DOUT), L11.4 (DIN)
- new net: L10.4 (DIN), L9.2 (DOUT)
- new net: L8.2 (DOUT), L9.4 (DIN)
- new net: L13.2 (DOUT), L14.4 (DIN)
- new net: L12.2 (DOUT), L13.4 (DIN)
- new net: L11.2 (DOUT), L12.4 (DIN)
- new net: L3.2 (DOUT), L4.4 (DIN)
- new net: L2.2 (DOUT), L3.4 (DIN)
- new net: L7.2 (DOUT), L8.4 (DIN)
- new net: L4.2 (DOUT), L5.4 (DIN)
- new net: L14.2 (DOUT), L15.4 (DIN)
- new net: L5.2 (DOUT), L6.4 (DIN)
- new net: L6.2 (DOUT), L7.4 (DIN)
- new net: L19.2 (DOUT), L20.4 (DIN)
- new net: L18.2 (DOUT), L19.4 (DIN)
- new net: L15.2 (DOUT), L16.4 (DIN)

Commit message: after-review updates
Other:
- note added: "100nF"
Changed lines of the file:
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@@
 	(generator_version "9.0")
 	(paper "A4")
+	(text "100nF\n"
+		(exclude_from_sim no)
+		(at 192.024 -39.37 0)
+		(effects
+			(font
+				(size 1.27 1.27)
+			)
+		)
+	)
+	(text "100nF\n"
+		(exclude_from_sim no)
+		(at 110.998 -38.862 0)
+		(effects
+			(font
+				(size 1.27 1.27)
+			)
+		)
+	)
+	(text "100nF\n"
+		(exclude_from_sim no)
+		(at 233.426 -39.116 0)
+		(effects
+			(font
+				(size 1.27 1.27)
+			)
+		)
+	)
+	(text "100nF\n"
+		(exclude_from_sim no)
+		(at 29.718 -38.862 0)
+		(effects
+			(font
+				(size 1.27 1.27)
+			)
+		)
+	)
+	(text "100nF\n"
+		(exclude_from_sim no)
+		(at 152.146 -39.116 0)
+		(effects
+			(font
+				(size 1.27 1.27)
+			)
+		)
+	)
+	(text "100nF\n"
+		(exclude_from_sim no)
+		(at 294.132 -39.116 0)
+		(effects
+			(font
+				(size 1.27 1.27)
+			)
+		)
+	)
+	(text "100nF\n"
+		(exclude_from_sim no)
+		(at -10.668 -39.116 0)
+		(effects
+			(font
+				(size 1.27 1.27)
+			)
+		)
+	)
+	(text "100nF\n"
+		(exclude_from_sim no)
+		(at 9.906 -38.862 0)
+		(effects
+			(font
+				(size 1.27 1.27)
+			)
+		)
+	)
+	(text "100nF\n"
+		(exclude_from_sim no)
+		(at -30.226 -38.862 0)
+		(effects
+			(font
+				(size 1.27 1.27)
+			)
+		)
+	)
+	(text "100nF\n"
+		(exclude_from_sim no)
+		(at 172.466 -39.116 0)
+		(effects
+			(font
+				(size 1.27 1.27)
+			)
+		)
+	)
+	(text "100nF\n"
+		(exclude_from_sim no)
+		(at 90.932 -39.37 0)
+		(effects
+			(font
+				(size 1.27 1.27)
+			)
+		)
+	)
+	(text "100nF\n"
+		(exclude_from_sim no)
+		(at 334.264 -38.608 0)
+		(effects
+			(font
+				(size 1.27 1.27)
+			)
+		)
+	)
+	(text "100nF\n"
+		(exclude_from_sim no)
+		(at 355.6 -39.37 0)
+		(effects
+			(font
+				(size 1.27 1.27)
+			)
+		)
+	)
+	(text "100nF\n"
+		(exclude_from_sim no)
+		(at 70.866 -39.116 0)
+		(effects
+			(font
+				(size 1.27 1.27)
+			)
+		)
+	)
+	(text "100nF\n"
+		(exclude_from_sim no)
+		(at 213.614 -39.116 0)
+		(effects
+			(font
+				(size 1.27 1.27)
+			)
+		)
+	)
+	(text "100nF\n"
+		(exclude_from_sim no)
+		(at 50.038 -38.862 0)
+		(effects
+			(font
+				(size 1.27 1.27)
+			)
+		)
+	)
+	(text "100nF\n"
+		(exclude_from_sim no)
+		(at 274.574 -38.862 0)
+		(effects
+			(font
+				(size 1.27 1.27)
+			)
+		)
+	)
+	(text "100nF\n"
+		(exclude_from_sim no)
+		(at 314.198 -39.116 0)
+		(effects
+			(font
+				(size 1.27 1.27)
+			)
+		)
+	)
+	(text "100nF\n"
+		(exclude_from_sim no)
+		(at 131.572 -38.862 0)
+		(effects
+			(font
+				(size 1.27 1.27)
+			)
+		)
+	)
+	(text "100nF\n"
+		(exclude_from_sim no)
+		(at 253.492 -39.116 0)
+		(effects
+			(font
+				(size 1.27 1.27)
+			)
+		)
+	)
 	(junction
 		(at 196.85 -59.69)
